File: hardware/Daughterboard/Initial/Prototype/Initial project.sch (KiCad schematic (older format))
At the start: 51 parts, among them IC1 LPC1517JBD48, IC2 TJF1051T/3, IC3 MC33660BEF, IC4 LM393D, IC5 AP2204-5.0, J1 M081X08, J2 M02PTH, J3 1X021, J4 M081X08, J5 M10\"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

Commit message: PCB work
Parts:
- removed J1: M081X08, Initial project:1X08, symbol Initial_project-eagle-import:M081X08
- removed J2: M02PTH, Initial project:1X02, symbol Initial_project-eagle-import:M02PTH
- removed J5: M10\", Initial project:1X10, symbol Initial_project-eagle-import:M10"
- removed J6: M06SIP, Initial project:1X06, symbol Initial_project-eagle-import:M06SIP
- removed JP1: JP2Q, Initial project:JP2Q, symbol Initial_project-eagle-import:JP2Q
- added C14: 0.33uC, symbol Device:C
- added C15, C16: 22pF, symbol Device:C
- added C17: 0.1uC, symbol Device:C
- added J1: AVR-ISP-6, symbol Connector:AVR-ISP-6
- added U1: ATmega328-PU, Package_DIP:DIP-28_W7.62mm, symbol MCU_Microchip_ATmega:ATmega328-PU
- added U2: L7805, symbol Regulator_Linear:L7805
- added X2: 16MHZ, symbol Device:Crystal
Connections:
- net labels added: 5V, SC, SD, SI, SO, Vbatt
- wire segments 220 -> 275
